Commit message: Tune Gazebo servo model for sim-to-real control

File: config/mycobot_280_m5_adaptive_gripper_sim.urdf.xacro (robot description, xacro)
@@ -1,4 +1,8 @@
 <?xml version="1.0"?>
 <robot xmlns:xacro="http://www.ros.org/wiki/xacro" name="mycobot_280_pick">
+  <xacro:property name="joint_effort" value="56.0"/>
+  <xacro:property name="joint_velocity" value="2.792527"/>
+  <xacro:property name="joint_damping" value="0.0"/>
+  <xacro:property name="joint_friction" value="0.0"/>
   <xacro:macro name="simple_inertial" params="mass ixx iyy izz">
     <inertial>
@@ -10,5 +14,4 @@
   <xacro:macro name="sim_link_gazebo" params="link_name">
     <gazebo reference="${link_name}">
-      <gravity>false</gravity>
       <self_collide>false</self_collide>
     </gazebo>
@@ -31,5 +34,5 @@
     </link>
     <link name="joint1">
-      <xacro:simple_inertial mass="0.35" ixx="0.0006" iyy="0.0006" izz="0.0006"/>
+      <xacro:simple_inertial mass="0.12" ixx="0.000148" iyy="0.000148" izz="0.000096"/>
       <visual>
         <geometry>
@@ -46,5 +49,5 @@
     </link>
     <link name="joint2">
-      <xacro:simple_inertial mass="0.30" ixx="0.0005" iyy="0.0005" izz="0.0005"/>
+      <xacro:simple_inertial mass="0.19" ixx="0.000148" iyy="0.000148" izz="0.000096"/>
       <visual>
         <geometry>
@@ -61,5 +64,5 @@
     </link>
     <link name="joint3">
-      <xacro:simple_inertial mass="0.25" ixx="0.0004" iyy="0.0004" izz="0.0004"/>
+      <xacro:simple_inertial mass="0.16" ixx="0.000148" iyy="0.000148" izz="0.000096"/>
       <visual>
         <geometry>
@@ -76,5 +79,5 @@
     </link>
     <link name="joint4">
-      <xacro:simple_inertial mass="0.20" ixx="0.0003" iyy="0.0003" izz="0.0003"/>
+      <xacro:simple_inertial mass="0.124" ixx="0.000103" iyy="0.000103" izz="0.000096"/>
       <visual>
         <geometry>
@@ -91,5 +94,5 @@
     </link>
     <link name="joint5">
-      <xacro:simple_inertial mass="0.15" ixx="0.0002" iyy="0.0002" izz="0.0002"/>
+      <xacro:simple_inertial mass="0.11" ixx="0.000103" iyy="0.000103" izz="0.000096"/>
       <visual>
         <geometry>
@@ -106,5 +109,5 @@
     </link>
     <link name="joint6">
-      <xacro:simple_inertial mass="0.12" ixx="0.00015" iyy="0.00015" izz="0.00015"/>
+      <xacro:simple_inertial mass="0.0739" ixx="0.00006649" iyy="0.00006649" izz="0.000096"/>
       <visual>
         <geometry>
@@ -121,5 +124,5 @@
     </link>
     <link name="joint6_flange">
-      <xacro:simple_inertial mass="0.05" ixx="0.00008" iyy="0.00008" izz="0.00008"/>
+      <xacro:simple_inertial mass="0.035" ixx="0.0000149" iyy="0.0000149" izz="0.0000196"/>
       <visual>
         <geometry>
@@ -144,6 +147,6 @@
     <joint name="joint2_to_joint1" type="revolute">
       <axis xyz="0 0 1"/>
-      <limit effort="1000.0" lower="-2.9321" upper="2.9321" velocity="0"/>
-      <dynamics damping="1.0" friction="0.10"/>
+      <limit effort="${joint_effort}" lower="-2.9321" upper="2.9321" velocity="${joint_velocity}"/>
+      <dynamics damping="${joint_damping}" friction="${joint_friction}"/>
       <parent link="joint1"/>
       <child link="joint2"/>
@@ -152,6 +155,6 @@
     <joint name="joint3_to_joint2" type="revolute">
       <axis xyz="0 0 1"/>
-      <limit effort="1000.0" lower="-2.4434" upper="2.4434" velocity="0"/>
-      <dynamics damping="1.0" friction="0.10"/>
+      <limit effort="${joint_effort}" lower="-2.4434" upper="2.4434" velocity="${joint_velocity}"/>
+      <dynamics damping="${joint_damping}" friction="${joint_friction}"/>
       <parent link="joint2"/>
       <child link="joint3"/>
@@ -160,6 +163,6 @@
     <joint name="joint4_to_joint3" type="revolute">
       <axis xyz="0 0 1"/>
-      <limit effort="1000.0" lower="-2.6179" upper="2.6179" velocity="0"/>
-      <dynamics damping="0.8" friction="0.08"/>
+      <limit effort="${joint_effort}" lower="-2.6179" upper="2.6179" velocity="${joint_velocity}"/>
+      <dynamics damping="${joint_damping}" friction="${joint_friction}"/>
       <parent link="joint3"/>
       <child link="joint4"/>
@@ -168,6 +171,6 @@
     <joint name="joint5_to_joint4" type="revolute">
       <axis xyz="0 0 1"/>
-      <limit effort="1000.0" lower="-2.6179" upper="2.6179" velocity="0"/>
-      <dynamics damping="0.6" friction="0.06"/>
+      <limit effort="${joint_effort}" lower="-2.6179" upper="2.6179" velocity="${joint_velocity}"/>
+      <dynamics damping="${joint_damping}" friction="${joint_friction}"/>
       <parent link="joint4"/>
       <child link="joint5"/>
@@ -176,6 +179,6 @@
     <joint name="joint6_to_joint5" type="revolute">
       <axis xyz="0 0 1"/>
-      <limit effort="1000.0" lower="-2.7052" upper="2.7925" velocity="0"/>
-      <dynamics damping="0.4" friction="0.05"/>
+      <limit effort="${joint_effort}" lower="-2.7052" upper="2.7925" velocity="${joint_velocity}"/>
+      <dynamics damping="${joint_damping}" friction="${joint_friction}"/>
       <parent link="joint5"/>
       <child link="joint6"/>
@@ -184,6 +187,6 @@
     <joint name="joint6output_to_joint6" type="revolute">
       <axis xyz="0 0 1"/>
-      <limit effort="1000.0" lower="-3.14159" upper="3.14159" velocity="0"/>
-      <dynamics damping="0.3" friction="0.04"/>
+      <limit effort="${joint_effort}" lower="-3.14159" upper="3.14159" velocity="${joint_velocity}"/>
+      <dynamics damping="${joint_damping}" friction="${joint_friction}"/>
       <parent link="joint6"/>
       <child link="joint6_flange"/>
@@ -196,5 +199,5 @@
     </joint>
     <link name="gripper_base">
-      <xacro:simple_inertial mass="0.08" ixx="0.00008" iyy="0.00008" izz="0.00008"/>
+      <xacro:simple_inertial mass="0.07" ixx="0.000010725" iyy="0.000014392" izz="0.000018517"/>
       <visual>
         <geometry>
@@ -211,5 +214,5 @@
     </link>
     <link name="gripper_left1">
-      <xacro:simple_inertial mass="0.02" ixx="0.00001" iyy="0.00001" izz="0.00001"/>
+      <xacro:simple_inertial mass="0.007" ixx="0.000001" iyy="0.000001" izz="0.000001"/>
       <visual>
         <geometry>
@@ -226,5 +229,5 @@
     </link>
     <link name="gripper_left2">
-      <xacro:simple_inertial mass="0.02" ixx="0.00001" iyy="0.00001" izz="0.00001"/>
+      <xacro:simple_inertial mass="0.007" ixx="0.000001" iyy="0.000001" izz="0.000001"/>
       <visual>
         <geometry>
@@ -241,5 +244,5 @@
     </link>
     <link name="gripper_left3">
-      <xacro:simple_inertial mass="0.02" ixx="0.00001" iyy="0.00001" izz="0.00001"/>
+      <xacro:simple_inertial mass="0.007" ixx="0.000001" iyy="0.000001" izz="0.000001"/>
       <visual>
         <geometry>
@@ -256,5 +259,5 @@
     </link>
     <link name="gripper_right1">
-      <xacro:simple_inertial mass="0.02" ixx="0.00001" iyy="0.00001" izz="0.00001"/>
+      <xacro:simple_inertial mass="0.007" ixx="0.000001" iyy="0.000001" izz="0.000001"/>
       <visual>
         <geometry>
@@ -271,5 +274,5 @@
     </link>
     <link name="gripper_right2">
-      <xacro:simple_inertial mass="0.02" ixx="0.00001" iyy="0.00001" izz="0.00001"/>
+      <xacro:simple_inertial mass="0.007" ixx="0.000001" iyy="0.000001" izz="0.000001"/>
       <visual>
         <geometry>
@@ -286,5 +289,5 @@
     </link>
     <link name="gripper_right3">
-      <xacro:simple_inertial mass="0.02" ixx="0.00001" iyy="0.00001" izz="0.00001"/>
+      <xacro:simple_inertial mass="0.007" ixx="0.000001" iyy="0.000001" izz="0.000001"/>
       <visual>
         <geometry>
@@ -302,6 +305,6 @@
     <joint name="gripper_controller" type="revolute">
       <axis xyz="0 0 1"/>
-      <limit effort="1000.0" lower="-0.74" upper="0.15" velocity="0"/>
-      <dynamics damping="0.15" friction="0.03"/>
+      <limit effort="${joint_effort}" lower="-0.74" upper="0.15" velocity="${joint_velocity}"/>
+      <dynamics damping="${joint_damping}" friction="${joint_friction}"/>
       <parent link="gripper_base"/>
       <child link="gripper_left3"/>
@@ -310,6 +313,6 @@
     <joint name="gripper_base_to_gripper_left2" type="revolute">
       <axis xyz="0 0 1"/>
-      <limit effort="1000.0" lower="-0.8" upper="0.5" velocity="0"/>
-      <dynamics damping="0.12" friction="0.02"/>
+      <limit effort="${joint_effort}" lower="-0.8" upper="0.5" velocity="${joint_velocity}"/>
+      <dynamics damping="${joint_damping}" friction="${joint_friction}"/>
       <parent link="gripper_base"/>
       <child link="gripper_left2"/>
@@ -319,6 +322,6 @@
     <joint name="gripper_left3_to_gripper_left1" type="revolute">
       <axis xyz="0 0 1"/>
-      <limit effort="1000.0" lower="-0.5" upper="0.5" velocity="0"/>
-      <dynamics damping="0.12" friction="0.02"/>
+      <limit effort="${joint_effort}" lower="-0.5" upper="0.5" velocity="${joint_velocity}"/>
+      <dynamics damping="${joint_damping}" friction="${joint_friction}"/>
       <parent link="gripper_left3"/>
       <child link="gripper_left1"/>
@@ -328,6 +331,6 @@
     <joint name="gripper_base_to_gripper_right3" type="revolute">
       <axis xyz="0 0 1"/>
-      <limit effort="1000.0" lower="-0.15" upper="0.7" velocity="0"/>
-      <dynamics damping="0.12" friction="0.02"/>
+      <limit effort="${joint_effort}" lower="-0.15" upper="0.7" velocity="${joint_velocity}"/>
+      <dynamics damping="${joint_damping}" friction="${joint_friction}"/>
       <parent link="gripper_base"/>
       <child link="gripper_right3"/>
@@ -337,6 +340,6 @@
     <joint name="gripper_base_to_gripper_right2" type="revolute">
       <axis xyz="0 0 1"/>
-      <limit effort="1000.0" lower="-0.5" upper="0.8" velocity="0"/>
-      <dynamics damping="0.12" friction="0.02"/>
+      <limit effort="${joint_effort}" lower="-0.5" upper="0.8" velocity="${joint_velocity}"/>
+      <dynamics damping="${joint_damping}" friction="${joint_friction}"/>
       <parent link="gripper_base"/>
       <child link="gripper_right2"/>
@@ -346,6 +349,6 @@
     <joint name="gripper_right3_to_gripper_right1" type="revolute">
       <axis xyz="0 0 1"/>
-      <limit effort="1000.0" lower="-0.5" upper="0.5" velocity="0"/>
-      <dynamics damping="0.12" friction="0.02"/>
+      <limit effort="${joint_effort}" lower="-0.5" upper="0.5" velocity="${joint_velocity}"/>
+      <dynamics damping="${joint_damping}" friction="${joint_friction}"/>
       <parent link="gripper_right3"/>
       <child link="gripper_right1"/>

File: config/mycobot_280_pick.urdf.xacro (robot description, xacro)
@@ -21,51 +21,65 @@
     </hardware>
     <joint name="joint2_to_joint1">
-      <command_interface name="position"/>
+      <command_interface name="position">
+        <param name="min">-2.9321</param>
+        <param name="max">2.9321</param>
+      </command_interface>
       <state_interface name="position">
         <param name="initial_value">${initial_positions['joint2_to_joint1']}</param>
       </state_interface>
-      <state_interface name="velocity"/>
     </joint>
     <joint name="joint3_to_joint2">
-      <command_interface name="position"/>
+      <command_interface name="position">
+        <param name="min">-2.4434</param>
+        <param name="max">2.4434</param>
+      </command_interface>
       <state_interface name="position">
         <param name="initial_value">${initial_positions['joint3_to_joint2']}</param>
       </state_interface>
-      <state_interface name="velocity"/>
     </joint>
     <joint name="joint4_to_joint3">
-      <command_interface name="position"/>
+      <command_interface name="position">
+        <param name="min">-2.6179</param>
+        <param name="max">2.6179</param>
+      </command_interface>
       <state_interface name="position">
         <param name="initial_value">${initial_positions['joint4_to_joint3']}</param>
       </state_interface>
-      <state_interface name="velocity"/>
     </joint>
     <joint name="joint5_to_joint4">
-      <command_interface name="position"/>
+      <command_interface name="position">
+        <param name="min">-2.6179</param>
+        <param name="max">2.6179</param>
+      </command_interface>
       <state_interface name="position">
         <param name="initial_value">${initial_positions['joint5_to_joint4']}</param>
       </state_interface>
-      <state_interface name="velocity"/>
     </joint>
     <joint name="joint6_to_joint5">
-      <command_interface name="position"/>
+      <command_interface name="position">
+        <param name="min">-2.7052</param>
+        <param name="max">2.7925</param>
+      </command_interface>
       <state_interface name="position">
         <param name="initial_value">${initial_positions['joint6_to_joint5']}</param>
       </state_interface>
-      <state_interface name="velocity"/>
     </joint>
     <joint name="joint6output_to_joint6">
-      <command_interface name="position"/>
+      <command_interface name="position">
+        <param name="min">-3.14159</param>
+        <param name="max">3.14159</param>
+      </command_interface>
       <state_interface name="position">
         <param name="initial_value">${initial_positions['joint6output_to_joint6']}</param>
       </state_interface>
-      <state_interface name="velocity"/>
     </joint>
     <joint name="gripper_controller">
-      <command_interface name="position"/>
+      <command_interface name="position">
+        <param name="min">-0.74</param>
+        <param name="max">0.15</param>
+      </command_interface>
       <state_interface name="position">
         <param name="initial_value">${initial_positions['gripper_controller']}</param>
       </state_interface>
-      <state_interface name="velocity"/>
     </joint>
   </ros2_control>
@@ -76,5 +90,4 @@
       <robot_param_node>robot_state_publisher</robot_param_node>
       <controller_manager_name>controller_manager</controller_manager_name>
-      <position_proportional_gain>1.0</position_proportional_gain>
     </plugin>
   </gazebo>
